File: electronics/Lab_PowerSupply.sch (KiCad schematic (older format))
At the start: 4 parts

Commit message: Update on electronic, reorder folder structure
Parts:
- removed U?: IR2112PBF, symbol IR2112PBF
- added U?: IR2112PBF, symbol IR2112PBF
Connections:
- net +3V3: now also U?.9 (VDD)
- net GND: now also U?.11 (SD), U?.12 (LIN), U?.13 (VSS), U?.14 (NC3), U?.2 (COM), U?.4 (NC1), U?.8 (NC2)
- net IGBT_E: now also U?.5 (VS)
- net IGBT_G: now also U?.7 (HO)
- net RC2: now also U?.10 (HIN)
Changed lines of the file:
@@
 	6225 925  6225 975
 Wire Wire Line
-	3775 3025 7175 3025
+	7175 3025 3775 3025
 Wire Wire Line
-	7175 3025 7175 1625
+	7175 1625 7175 3025
 Wire Wire Line
 	7175 1625 7125 1625
@@
 $Comp
 L IR2112PBF U?
-U 1 1 59A02654
-P 1575 4000
-F 0 "U?" H 1825 3950 60  0000 C CNN
-F 1 "IR2112PBF" H 1825 5050 60  0000 C CNN
-F 2 "" H 1575 4000 60  0001 C CNN
-F 3 "" H 1575 4000 60  0001 C CNN
-	1    1575 4000
+U 1 1 59A2B388
+P 1200 4000
+F 0 "U?" H 1500 3950 60  0000 C CNN
+F 1 "IR2112PBF" H 1500 5050 60  0000 C CNN
+F 2 "" H 1250 4000 60  0001 C CNN
+F 3 "" H 1250 4000 60  0001 C CNN
+	1    1200 4000
 	1    0    0    -1
 $EndComp
 Wire Wire Line
-	1375 3950 1325 3950
+	1000 3750 950  3750
 Wire Wire Line
-	1325 3750 1325 4000
+	950  3950 1000 3950
 Wire Wire Line
-	1325 3750 1375 3750
+	1000 3850 950  3850
+Connection ~ 950  3850
 Wire Wire Line
-	1375 3850 1325 3850
-Connection ~ 1325 3850
+	2000 3750 2050 3750
+Wire Wire Line
+	2050 3850 2000 3850
+Connection ~ 2050 3850
+Wire Wire Line
+	950  3450 950  4000
 $Comp
 L GND #PWR?
-U 1 1 59A027EB
-P 1325 4000
-F 0 "#PWR?" H 1325 3750 50  0001 C CNN
-F 1 "GND" H 1325 3850 50  0000 C CNN
-F 2 "" H 1325 4000 50  0000 C CNN
-F 3 "" H 1325 4000 50  0000 C CNN
-	1    1325 4000
+U 1 1 59A2B7AF
+P 950 4000
+F 0 "#PWR?" H 950 3750 50  0001 C CNN
+F 1 "GND" H 950 3850 50  0000 C CNN
+F 2 "" H 950 4000 50  0001 C CNN
+F 3 "" H 950 4000 50  0001 C CNN
+	1    950  4000
 	1    0    0    -1
 $EndComp
-Connection ~ 1325 3950
-Wire Wire Line
-	2275 3750 2325 3750
-Wire Wire Line
-	2325 3750 2325 4000
-Wire Wire Line
-	2325 3850 2275 3850
 $Comp
 L GND #PWR?
-U 1 1 59A0293F
-P 2325 4000
-F 0 "#PWR?" H 2325 3750 50  0001 C CNN
-F 1 "GND" H 2325 3850 50  0000 C CNN
-F 2 "" H 2325 4000 50  0000 C CNN
-F 3 "" H 2325 4000 50  0000 C CNN
-	1    2325 4000
+U 1 1 59A2B82F
+P 2050 4000
+F 0 "#PWR?" H 2050 3750 50  0001 C CNN
+F 1 "GND" H 2050 3850 50  0000 C CNN
+F 2 "" H 2050 4000 50  0001 C CNN
+F 3 "" H 2050 4000 50  0001 C CNN
+	1    2050 4000
 	1    0    0    -1
 $EndComp
-Connection ~ 2325 3850
 $Comp
 L +3V3 #PWR?
-U 1 1 59A02AB3
-P 1325 3000
-F 0 "#PWR?" H 1325 2850 50  0001 C CNN
-F 1 "+3V3" H 1325 3140 50  0000 C CNN
-F 2 "" H 1325 3000 50  0000 C CNN
-F 3 "" H 1325 3000 50  0000 C CNN
-	1    1325 3000
+U 1 1 59A2B8C6
+P 950 3000
+F 0 "#PWR?" H 950 2850 50  0001 C CNN
+F 1 "+3V3" H 950 3140 50  0000 C CNN
+F 2 "" H 950 3000 50  0001 C CNN
+F 3 "" H 950 3000 50  0001 C CNN
+	1    950  3000
 	1    0    0    -1
 $EndComp
+Text Label 2050 3050 0    60   ~ 0
+IGBT_G
 Wire Wire Line
-	1375 3050 1325 3050
+	2050 3050 2000 3050
 Wire Wire Line
-	1325 3050 1325 3000
+	1000 3050 950  3050
+Wire Wire Line
+	950  3050 950  3000
+Connection ~ 950  3950
+Wire Wire Line
+	2050 3750 2050 4000
+Text Label 950  3350 2    60   ~ 0
+RC2
+Text Label 2050 3350 0    60   ~ 0
+IGBT_E
+Wire Wire Line
+	950  3350 1000 3350
+Wire Wire Line
+	2000 3350 2050 3350
+Wire Wire Line
+	1000 3550 950  3550
+Connection ~ 950  3750
+Wire Wire Line
+	1000 3450 950  3450
+Connection ~ 950  3550
 $EndSCHEMATC
